File: sample-project/sample-project.kicad_pcb (KiCad board)
At the start: 2 copper layers, 5 parts

Commit message: New connectors
Parts:
- added REF**: RCA-105A, Pakequis_Footprints:RCA-105A, F.Cu at (165.1, 121.9)
- added REF**: RCA-105, Pakequis_Footprints:RCA-105, F.Cu at (165.1, 66.0)
- added REF**: RCA-105-105A, Pakequis_Footprints:RCA-105-105A, F.Cu at (165.1, 94.0)
- added REF**: PJ-320A, Pakequis_Footprints:PJ-320A, F.Cu at (147.3, 58.4)
- moved REF** 25.1 mm to (119.4, 91.4)
- moved REF** 25.1 mm to (83.8, 91.4)
- moved REF** 25.1 mm to (83.8, 58.4)
- moved REF** 25.1 mm to (119.4, 81.3)
- moved REF** 25.1 mm to (129.5, 58.4)
Other:
- board outline added: 127 x 88.9 mm
